File: linebot/kicad/linebot.sch (KiCad schematic (older format))
At the start: 14 parts, among them IC1 ATTINY85-P, P1 Motor, P2 Motor, Q1 BC817-40, Q2 BC817-40, Q3 PT, Q4 PT

Commit message: Added second project
Parts:
- removed Q3, Q4: PT, LEDs:LED-5MM, symbol PHOTO_TRANSISTOR
- added U1, U2: Phototransistor, LEDs:LED-5MM, symbol Phototransistor
- BT1: footprint mybattery:Batterie_aufrecht -> mybattery:batteryholder_AAAx2
Connections:
- wire segments 13 -> 17
Changed lines of the file:
@@
 LIBS:valves
 LIBS:PHOTO_TRANSISTOR
+LIBS:phototransistor
 LIBS:linebot-cache
 EELAYER 25 0
@@
 P 4600 3150
 F 0 "IC1" H 3450 3550 50  0000 C CNN
-F 1 "ATTINY85-P" H 4600 3550 50  0000 C CNN
-F 2 "Housings_DIP:DIP-8_W7.62mm" H 5050 2850 50  0000 C CIN
+F 1 "ATTINY85-P" H 5300 3150 50  0000 C CNN
+F 2 "Housings_DIP:DIP-8_W7.62mm" H 5050 2850 50  0001 C CIN
 F 3 "" H 4600 3150 50  0000 C CNN
 	1    4600 3150
@@
 F 3 "" H 5950 2900 50  0000 C CNN
 	1    5950 2900
-	1    0    0    -1
-$EndComp
-$Comp
-L PHOTO_TRANSISTOR Q3
-U 1 1 587788A7
-P 1700 2900
-F 0 "Q3" V 1540 2900 60  0000 C CNN
-F 1 "PT" V 1860 2900 60  0000 C CNN
-F 2 "LEDs:LED-5MM" H 1700 2900 60  0001 C CNN
-F 3 "" H 1700 2900 60  0000 C CNN
-	1    1700 2900
 	1    0    0    -1
 $EndComp
@@
 $EndComp
 $Comp
-L PHOTO_TRANSISTOR Q4
-U 1 1 58778D19
-P 2200 3550
-F 0 "Q4" V 2040 3550 60  0000 C CNN
-F 1 "PT" V 2360 3550 60  0000 C CNN
-F 2 "LEDs:LED-5MM" H 2200 3550 60  0001 C CNN
-F 3 "" H 2200 3550 60  0000 C CNN
-	1    2200 3550
-	1    0    0    -1
-$EndComp
-$Comp
 L R R4
 U 1 1 58778D1F
@@
 	1    0    0    -1
 $EndComp
-Wire Wire Line
-	1750 3100 3250 3100
 Wire Wire Line
 	2500 3750 2250 3750
@@
 	1    0    0    -1
 $EndComp
-Wire Wire Line
-	2200 2350 2200 3200
-Wire Wire Line
-	2200 3200 3250 3200
 $Comp
 L GND #PWR012
@@
 F 0 "BT1" H 6300 3200 50  0000 L CNN
 F 1 "Battery" H 6300 3100 50  0000 L CNN
-F 2 "mybattery:Batterie_aufrecht" V 6200 3190 50  0001 C CNN
+F 2 "mybattery:batteryholder_AAAx2" V 6200 3190 50  0001 C CNN
 F 3 "" V 6200 3190 50  0000 C CNN
 	1    6200 3150
 	1    0    0    -1
 $EndComp
+Wire Wire Line
+	3250 3200 2500 3200
+Wire Wire Line
+	2500 3200 2500 3100
+Wire Wire Line
+	2500 3100 1750 3100
+Wire Wire Line
+	3250 3100 2900 3100
+Wire Wire Line
+	2900 3100 2900 2500
+Wire Wire Line
+	2900 2500 2200 2500
+Wire Wire Line
+	2200 2500 2200 2350
+$Comp
+L Phototransistor U1
+U 1 1 58B8213F
+P 1750 2900
+F 0 "U1" H 1920 2830 60  0000 C CNN
+F 1 "Phototransistor" V 1500 2900 60  0000 C CNN
+F 2 "LEDs:LED-5MM" H 1730 2900 60  0001 C CNN
+F 3 "" H 1730 2900 60  0001 C CNN
+	1    1750 2900
+	1    0    0    -1
+$EndComp
+$Comp
+L Phototransistor U2
+U 1 1 58B821B4
+P 2250 3550
+F 0 "U2" H 2420 3480 60  0000 C CNN
+F 1 "Phototransistor" V 2000 3550 60  0000 C CNN
+F 2 "LEDs:LED-5MM" H 2230 3550 60  0001 C CNN
+F 3 "" H 2230 3550 60  0001 C CNN
+	1    2250 3550
+	1    0    0    -1
+$EndComp

Commit message: Boards updated
Parts:
- removed Q1, Q2: BC817-40, TO_SOT_Packages_THT:TO-92_Inline_Narrow_Oval, symbol BC817-40
- added C1: 10u, Capacitors_ThroughHole:C_Rect_L13_W6_H12_P10, symbol CP
- added D2, D3: 1N4148, Diodes_ThroughHole:Diode_DO-35_SOD27_Horizontal_RM10, symbol D
- added SW1: Switch, schiebeschalter:Schiebeschalter, symbol Switch
- added U3, U4: BC337, BC337:BC337_narrow, symbol BC337
- R5: value 330 -> 220
Connections:
- net GND: now also C1.2, U3.3 (E), U4.3 (E)
- net VCC: now also C1.1, D2.1 (K), D3.1 (K), SW1.2; no longer BT1.1
- net at IC1.6 (PB1(MISO/DO/AIN1/OC0B/OC1A/PCINT1)): now also R1.2; no longer R5.1
- net at IC1.7 (PB2(SCK/USCK/SCL/T0/INT0/ADC1/PCINT2)): now also R5.1; no longer R1.2
- net at P1.1 (P1): now also D2.2 (A), U3.1 (C)
- net at R1.1: now also U3.2 (B)
- net at P2.1 (P1): now also D3.2 (A), U4.1 (C)
- net at R2.1: now also U4.2 (B)
- new net: BT1.1, SW1.1
Other:
- moved on the sheet: BT1, P2, R2
